File: Support Board/support_board/power.kicad_sch (KiCad schematic)
At the start: 51 parts, among them J1 Conn_01x02_Socket, J2 Conn_01x02_Socket, J3 Conn_01x02_Socket, J4 Conn_01x02_Socket, J505 Conn_01x01_Socket, J6 CURRENT_SENSE_TAP, J8 VOLTAGE_SENSE_TAP, U503 INA169, U504 MCP6002T-E/OT

Commit message: Updated PM files and Schematics in the Support Board
Changed lines of the file:
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@@
 	)
 	(junction
-		(at 125.73 104.14)
+		(at 60.96 149.86)
 		(diameter 0)
 		(color 0 0 0 0)
 	)
 	(junction
-		(at 60.96 149.86)
+		(at 125.73 104.14)
 		(diameter 0)
 		(color 0 0 0 0)
@@
 	(wire
 		(pts
-			(xy 60.96 149.86) (xy 72.39 149.86)
-		)
-		(stroke
-			(width 0)
-			(type default)
-		)
-	)
-	(wire
-		(pts
 			(xy 119.38 38.1) (xy 123.19 38.1)
 		)
@@
 	(wire
 		(pts
+			(xy 60.96 149.86) (xy 71.12 149.86)
+		)
+		(stroke
+			(width 0)
+			(type default)
+		)
+	)
+	(wire
+		(pts
 			(xy 166.37 60.96) (xy 166.37 53.34)
 		)
@@
 		(dnp no)
 		(fields_autoplaced yes)
-		(property "Reference" "#FLG01"
+		(property "Reference" "#FLG0101"
 			(at 212.725 49.53 0)
 			(effects
@@
 			(project "support_board"
 				(path "/a27a0383-1f9a-4fd1-ac31-ce73f638ee85/82bbc2ed-b886-483f-9163-240e584b498f"
-					(reference "#FLG01")
+					(reference "#FLG0101")
 					(unit 1)
 				)
