File: Support Board/support_board/switch.kicad_sch (KiCad schematic)
At the start: 3 parts

Commit message: Updated PM files and Schematics in the Support Board
Parts:
- D201: footprint LED_SMD:LED_0603_1608Metric -> LED_SMD:LED_0402_1005Metric_Pad0.77x0.64mm_HandSolder
Changed lines of the file:
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@@
 			)
 		)
-		(property "Footprint" "LED_SMD:LED_0603_1608Metric"
+		(property "Footprint" "LED_SMD:LED_0402_1005Metric_Pad0.77x0.64mm_HandSolder"
 			(at 53.34 80.01 0)
 			(effects
